File: SkeleKatze/pcb/SkeleKatze.kicad_sch (KiCad schematic)
At the start: 6 parts, among them SW2 SW_Push

Commit message: Updated base image to fix mask issues
Parts:
- Lg1: footprint SkeleKatze-Lib:SkeleKatze-Merged-NFS -> SkeleKatze-Lib:SkeleKatze-R2.0
Changed lines of the file:
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@@
 			)
 		)
-		(property "Footprint" "SkeleKatze-Lib:SkeleKatze-Merged-NFS"
+		(property "Footprint" "SkeleKatze-Lib:SkeleKatze-R2.0"
 			(at 120.65 73.66 0)
 			(hide yes)
